Commit message: init development

File: hexapod_description/urdf/reignblaze_model.xacro (robot description, xacro)
@@ -51,5 +51,5 @@
 	</gazebo>
 	<!-- Head Pan and Tilt properties -->
-	<joint name="head_pan_joint" type="revolute">
+	<joint name="pan_joint" type="fixed">
 		<parent link="body_link"/>
 		<child link="head_pan_link"/>
@@ -68,5 +68,5 @@
 		</inertial>
 	</link>
-	<joint name="head_tilt_joint" type="revolute">
+	<joint name="tilt_joint" type="fixed">
 		<parent link="head_pan_link"/>
 		<child link="head_tilt_link"/>

Commit message: enable teleop twist keyboard & gazebo

File: hexapod_description/urdf/reignblaze_model.xacro (robot description, xacro)
@@ -21,5 +21,5 @@
 	<link name="body_link">
 		<visual>
-	  		<origin xyz="0.0 0.0 0.0" rpy="${pi/2} 0.0 0.0" />
+	  		<origin xyz="0.0 0.0 -0.01925" rpy="${pi/2} 0.0 0.0" />
 			<geometry>
 				<mesh filename="package://hexapod_description/meshes/reignblaze/body.stl" scale="0.001 0.001 0.001"/>
@@ -30,5 +30,5 @@
 		</visual>
 		<collision>
-			<origin xyz="0.0 0.0 0.0" rpy="${pi/2} 0.0 0.0"/>
+			<origin xyz="0.0 0.0 -0.01925" rpy="${pi/2} 0.0 0.0"/>
 			<geometry>
 				<box size="0.27 0.09 0.138" />
@@ -39,5 +39,5 @@
 		</collision>
 		<inertial>
-			<origin xyz="0.0 0.0 0.0" rpy="${pi/2} 0.0 0.0" />
+			<origin xyz="0.0 0.0 -0.01925" rpy="${pi/2} 0.0 0.0" />
 			<mass value="0.00001"/>
 			<inertia

Commit message: enable gazebo

File: hexapod_description/urdf/reignblaze_model.xacro (robot description, xacro)
@@ -1,8 +1,9 @@
 <?xml version="1.0" encoding="UTF-8" ?>
 <robot xmlns:xacro="http://ros.org/wiki/xacro" name="reignblaze">
+	<xacro:include filename="accessories/reignblaze_accessories.xacro" />
 	<!-- parameters -->
 	<xacro:property name="pi" value="3.1415926535897931" />
-	<xacro:property name="body_length_x" value="0.250" />
-	<xacro:property name="body_length_y" value="0.125" />
+	<xacro:property name="body_length_x" value="0.27" />
+	<xacro:property name="body_length_y" value="0.09" />
 	<xacro:property name="coxa_length" value="0.044" />
 	<xacro:property name="femur_length" value="0.0545" />
@@ -13,6 +14,12 @@
 		</plugin>
 	</gazebo>
+	<link name="base_footprint"/>
+	<joint name="base_joint" type="fixed">
+		<parent link="base_footprint"/>
+		<child link="base_link"/>
+		<origin xyz="0 0 0" rpy="0 0 0"/>
+	</joint>
 	<link name="base_link"/>
-	<joint name="base_joint" type="fixed">
+	<joint name="body_joint" type="fixed">
 		<parent link="base_link" />
 		<child link="body_link" />
@@ -21,138 +28,48 @@
 	<link name="body_link">
 		<visual>
-	  		<origin xyz="0.0 0.0 -0.01925" rpy="${pi/2} 0.0 0.0" />
+	  		<origin xyz="0.0 0.0 0.0" rpy="${pi/2} 0.0 0.0" />
 			<geometry>
 				<mesh filename="package://hexapod_description/meshes/reignblaze/body.stl" scale="0.001 0.001 0.001"/>
 			</geometry>
-			<material name="">
-				<color rgba="0.7 0.7 0.7 1" />
+			<material name="white">
+				<color rgba="1.0 1.0 1.0 1.0"/>
 			</material>
 		</visual>
 		<collision>
-			<origin xyz="0.0 0.0 -0.01925" rpy="${pi/2} 0.0 0.0"/>
+			<origin xyz="0.0 0.0 0.04225" rpy="0.0 0.0 0.0"/>
 			<geometry>
-				<box size="0.27 0.09 0.138" />
+				<box size="${body_length_x} ${body_length_y} 0.121" />
 			</geometry>
-			<material name="">
-				<color rgba="0.7 0.7 0.7 1"/>
+			<material name="acrylic">
+				<color rgba="0.9 0.9 1.0 0.6"/>
 			</material>
 		</collision>
 		<inertial>
-			<origin xyz="0.0 0.0 -0.01925" rpy="${pi/2} 0.0 0.0" />
-			<mass value="0.00001"/>
+			<origin xyz="0.0 0.0 0.0" rpy="0.0 0.0 0.0" />
+			<mass value="0.84"/>
 			<inertia
-			ixx="1.0" ixy="0.0"  ixz="0.0"
-			iyy="1.0" iyz="0.0"
-			izz="1.0" />
+			ixx="0.001592" ixy="0.0"  ixz="0.0"
+			iyy="0.006128" iyz="0.0"
+			izz="0.005670" />
 		</inertial>
 	</link>
 	<gazebo reference="body_link">
-		<material>Gazebo/DarkGrey</material>
+		<material>Gazebo/White</material>
 	</gazebo>
-	<!-- Head Pan and Tilt properties -->
-	<joint name="head_pan_joint" type="revolute">
-		<parent link="body_link"/>
-		<child link="head_pan_link"/>
-		<axis xyz="0.0 0.0 1.0" />
-		<origin xyz="0.145 0.0 0.080" />
-		<limit lower="-${3.14}" upper="${3.14}" effort="10000" velocity="100" />
-	</joint>
-	<link name="head_pan_link">
-		<inertial>
-		    	<origin xyz="0.0 0.0 0.0" rpy="0.0 0.0 0.0" />
-		    	<mass value="0.00001"/>
-		    	<inertia
-			ixx="1.0" ixy="0.0"  ixz="0.0"
-			iyy="1.0" iyz="0.0"
-			izz="1.0" />
-		</inertial>
-	</link>
-	<joint name="head_tilt_joint" type="revolute">
-		<parent link="head_pan_link"/>
-		<child link="head_tilt_link"/>
-		<axis xyz="0.0 1.0 0.0" />
-		<origin xyz="0.0 0.0 0.020" />
-		<limit lower="-${3.14}" upper="${3.14}" effort="10000" velocity="100" />
-	</joint>
-	<link name="head_tilt_link">
-		<inertial>
-			<origin xyz="0.0 0.0 0.0" rpy="0.0 0.0 0.0" />
-			<mass value="0.00001"/>
-			<inertia
-			ixx="1.0" ixy="0.0"  ixz="0.0"
-			iyy="1.0" iyz="0.0"
-			izz="1.0" />
-		</inertial>
-	</link>
-	<!-- Camera properties -->
-	<joint name="camera_rgb_joint" type="fixed">
-		<parent link="head_tilt_link" />
-		<child link="camera_rgb_optical_frame" />
-		<origin xyz="0.0 0.0 0.0" rpy="${pi/2} ${pi} ${pi/2}" />
-	</joint>
-	<link name="camera_rgb_optical_frame">
-		<inertial>
-			<origin xyz="0.0 0.0 0.0" rpy="0.0 0.0 0.0" />
-			<mass value="0.00001"/>
-			<inertia
-			ixx="1.0" ixy="0.0"  ixz="0.0"
-			iyy="1.0" iyz="0.0"
-			izz="1.0" />
-		</inertial>
-	</link>
-	<joint name="camera_depth_joint" type="fixed">
-		<parent link="head_tilt_link" />
-		<child link="camera_depth_optical_frame" />
-		<origin xyz="0.0 0.0 0.0" rpy="${pi/2} ${pi} ${pi/2}" />
-	</joint>
-	<link name="camera_depth_optical_frame" >
-		<inertial>
-			<origin xyz="0.0 0.0 0.0" rpy="0.0 0.0 0.0" />
-			<mass value="0.00001"/>
-			<inertia
-			ixx="1.0" ixy="0.0"  ixz="0.0"
-			iyy="1.0" iyz="0.0"
-			izz="1.0" />
-		</inertial>
-	</link>
-	<joint name="camera_depth_frame" type="fixed">
-		<parent link="head_tilt_link" />
-		<child link="camera_depth_frame_link" />
-		<origin xyz="0.0 0.0 0.0" />
-	</joint>
-	<link name="camera_depth_frame_link" >
-		<inertial>
-			<origin xyz="0.0 0.0 0.0" rpy="0.0 0.0 0.0" />
-			<mass value="0.00001"/>
-			<inertia
-			ixx="1.0" ixy="0.0"  ixz="0.0"
-			iyy="1.0" iyz="0.0"
-			izz="1.0" />
-		</inertial>
-	</link>
-	<!-- IMU properties -->
-	<joint name="imu_joint" type="fixed">
-		<parent link="base_link" />
-		<child link="imu_link" />
-		<origin xyz="0.0 0.0 0.0" rpy="0.0 0.0 0.0" />
-	</joint>
-	<link name="imu_link">
-		<inertial>
-			<origin xyz="0.0 0.0 0.0" rpy="0.0 0.0 0.0" />
-			<mass value="0.00001"/>
-			<inertia
-			ixx="1.0" ixy="0.0"  ixz="0.0"
-			iyy="1.0" iyz="0.0"
-			izz="1.0" />
-		</inertial>
-	</link>
 	<!-- Joint properties -->
-	<xacro:property name="joint_lower_limit" value="-${3.14}" />
-	<xacro:property name="joint_upper_limit" value="${3.14}" />
+	<xacro:property name="joint_lower_limit" value="-${pi}" />
+	<xacro:property name="joint_upper_limit" value="${pi}" />
 	<xacro:property name="joint_effort" value="6.0" />
 	<xacro:property name="joint_velocity" value="0.524" />
+	<!--
+	<xacro:property name="joint_lower_limit" value="-2.6179939" />
+	<xacro:property name="joint_upper_limit" value="2.6179939" />
+	<xacro:property name="joint_effort" value="2.8" />
+	<xacro:property name="joint_velocity" value="5.6548668" />
+	-->
 	<!-- Leg macro -->
 	<xacro:macro name="leg" params="side position x y angle axis">
 		<!-- leg position -->
+		<!--
 		<joint name="leg_center_joint_${side}${position}" type="fixed">
 			<origin xyz="${x} ${y} 0.0" rpy="0.0 0.0 0.0" />
@@ -163,15 +80,16 @@
 			<inertial>
 				<origin xyz="0.0 0.0 0.0" rpy="0.0 0.0 0.0" />
-				<mass value="0.00001"/>
-				<inertia
-				ixx="1.0" ixy="0.0"  ixz="0.0"
-				iyy="1.0" iyz="0.0"
-				izz="1.0" />
-			</inertial>
-		</link>
+				<mass value="0.000001"/>
+				<inertia
+					ixx="0.0" ixy="0.0" ixz="0.0"
+					iyy="0.0" iyz="0.0"
+					izz="0.0"/>
+			</inertial>
+		</link>
+		-->
 		<!-- coxa -->
 		<joint name="coxa_joint_${side}${position}" type="revolute">
-			<origin xyz="0.0 0.0 0.0" rpy="0.0 0.0 ${angle}" />
-			<parent link="leg_center_${side}${position}" />
+			<origin xyz="${x} ${y} 0.0" rpy="0.0 0.0 ${angle}" />
+			<parent link="body_link" />
 			<child link="coxa_${side}${position}" />
 			<axis xyz="0.0 0.0 1.0" />
@@ -190,32 +108,34 @@
 		<link name="coxa_${side}${position}">
 			<visual>
-				<origin xyz="0.0 0.0 0.0" rpy="${pi/2} 0.0 ${pi/2}"/>
+				<origin xyz="0.0 0.0 0.0" rpy="0.0 0.0 ${pi/2}"/>
 				<geometry>
 					<mesh filename="package://hexapod_description/meshes/reignblaze/coxa.stl" scale="0.001 0.001 0.001"/>
 				</geometry>
-				<material name="">
-					<color rgba="0.7 0.7 0.7 1"/>
+				<material name="black">
+					<color rgba="0.0 0.0 0.0 1.0"/>
 				</material>
 			</visual>
-			<collision>
-				<origin xyz="0.0 0.0 0.0" rpy="${pi/2} 0.0 ${pi/2}" />
-				<geometry>
-					<mesh filename="package://hexapod_description/meshes/reignblaze/coxa.stl" scale="0.001 0.001 0.001"/>
-				</geometry>
-				<material name="">
-					<color rgba="0.7 0.7 0.7 1" />
-				</material>
-			</collision>
-			<inertial>
-				<origin xyz="0.0 0.0 0.0" rpy="${pi/2} 0.0 ${pi/2}" />
-				<mass value="0.00001"/>
-				<inertia
-				ixx="1.0" ixy="0.0"  ixz="0.0"
-				iyy="1.0" iyz="0.0"
-				izz="1.0" />
+			<!--
+			<collision>
+				<origin xyz="-0.00225 0.0 0.0" rpy="0.0 0.0 0.0" />
+				<geometry>
+					<box size="0.0275 0.032 0.040"/>
+				</geometry>
+				<material name="acrylic">
+					<color rgba="0.9 0.9 1.0 0.6"/>
+				</material>
+			</collision>
+			-->
+			<inertial>
+				<origin xyz="-0.00225 0.0 0.0" rpy="0.0 0.0 0.0" />
+				<mass value="0.056"/>
+				<inertia
+				ixx="0.000012245" ixy="0.0"  ixz="0.0"
+				iyy="0.000010996" iyz="0.0"
+				izz="0.000008308" />
 		    </inertial>
 		</link>
 		<gazebo reference="coxa_${side}${position}">
-			<material>Gazebo/DarkGrey</material>
+			<material>Gazebo/Black</material>
 		</gazebo>
 		<!-- femur -->
@@ -243,24 +163,41 @@
 					<mesh filename="package://hexapod_description/meshes/reignblaze/femur.stl" scale="0.001 0.001 0.001"/>
 				</geometry>
-				<material name="">
-					<color rgba="0.7 0.7 0.7 1"/>
+				<material name="dark">
+					<color rgba="0.3 0.3 0.3 1.0"/>
 				</material>
 			</visual>
 		    	<collision>
-				<origin xyz="0.0 0.0 0.0" rpy="0.0 -${pi/2} ${pi/2}" />
-				<geometry>
-					<mesh filename="package://hexapod_description/meshes/reignblaze/femur.stl" scale="0.001 0.001 0.001"/>
-				</geometry>
-				<material name="">
-					<color rgba="0.7 0.7 0.7 1" />
-				</material>
-			</collision>
-			<inertial>
-				<origin xyz="0.0 0.0 0.0" rpy="0.0 -${pi/2} ${pi/2}" />
-				<mass value="0.00001"/>
-				<inertia
-				ixx="1.0" ixy="0.0"  ixz="0.0"
-				iyy="1.0" iyz="0.0"
-				izz="1.0" />
+				<origin xyz="0.0 -0.0135 0.0" rpy="0.0 0.0 0.0" />
+				<geometry>
+					<box size="0.032 0.050 0.040"/>
+				</geometry>
+				<material name="acrylic">
+					<color rgba="0.9 0.9 1.0 0.6"/>
+				</material>
+			</collision>
+			<collision>
+				<origin xyz="-0.0135 -0.0545 0.0" rpy="0.0 0.0 0.0" />
+				<geometry>
+					<box size="0.050 0.032 0.040"/>
+				</geometry>
+				<material name="acrylic">
+					<color rgba="0.9 0.9 1.0 0.6"/>
+				</material>
+			</collision>
+			<inertial>
+				<origin xyz="0.0 -0.0135 0.0" rpy="0.0 0.0 0.0" />
+				<mass value="0.056"/>
+				<inertia
+				ixx="0.000019133" ixy="0.0"  ixz="0.0"
+				iyy="0.000012245" iyz="0.0"
+				izz="0.000016445" />
+			</inertial>
+			<inertial>
+				<origin xyz="-0.0135 -0.0545 0.0" rpy="0.0 0.0 0.0" />
+				<mass value="0.056"/>
+				<inertia
+				ixx="0.000012245" ixy="0.0"  ixz="0.0"
+				iyy="0.000019133" iyz="0.0"
+				izz="0.000016445" />
 			</inertial>
 		</link>
@@ -273,5 +210,5 @@
 			<parent link="femur_${side}${position}" />
 			<child link="tibia_${side}${position}" />
-			<axis xyz="0.0 0.0 ${axis}" />
+			<axis xyz="0.0 0.0 ${-axis}" />
 			<limit lower="${joint_lower_limit}" upper="${joint_upper_limit}" effort="${joint_effort}" velocity="${joint_velocity}" />
 		</joint>
@@ -288,40 +225,49 @@
 		<link name="tibia_${side}${position}">
 			<visual>
-				<origin xyz="0.0 0.0 0.0" rpy="${pi/2} -${pi/2} 0.0"/>
+				<origin xyz="0.0 0.0 0.0" rpy="0.0 ${pi/2} ${pi/2}"/>
 				<geometry>
 					<mesh filename="package://hexapod_description/meshes/reignblaze/tibia.stl" scale="0.001 0.001 0.001"/>
 				</geometry>
-				<material name="">
-					<color rgba="0.7 0.7 0.7 1"/>
+				<material name="black">
+					<color rgba="0.0 0.0 0.0 1.0"/>
 				</material>
 			</visual>
 			<collision>
-				<origin xyz="0.0 0.0 0.0" rpy="${pi/2} -${pi/2} 0.0" />
-				<geometry>
-					<mesh filename="package://hexapod_description/meshes/reignblaze/tibia.stl" scale="0.001 0.001 0.001"/>
-				</geometry>
-				<material name="">
-					<color rgba="0.7 0.7 0.7 1" />
-				</material>
-			</collision>
-			<inertial>
-				<origin xyz="0.0 0.0 0.0" rpy="${pi/2} -${pi/2} 0.0" />
-				<mass value="0.00001"/>
-				<inertia
-				ixx="1.0" ixy="0.0"  ixz="0.0"
-				iyy="1.0" iyz="0.0"
-				izz="1.0" />
+				<origin xyz="0.0516 0.0 0.0" rpy="0.0 0.0 0.0" />
+				<geometry>
+					<box size="0.065 0.01 0.0475"/>
+				</geometry>
+				<material name="acrylic">
+					<color rgba="0.9 0.9 1.0 0.6"/>
+				</material>
+			</collision>
+			<collision>
+				<origin xyz="0.0967 0.0 0.0" rpy="0.0 ${pi/2} 0.0" />
+				<geometry>
+					<sphere radius="0.0071"/>
+				</geometry>
+				<material name="acrylic">
+					<color rgba="0.9 0.9 1.0 0.6"/>
+				</material>
+			</collision>
+			<inertial>
+				<origin xyz="0.0516 0.0 0.0" rpy="0.0 0.0 0.0" />
+				<mass value="0.014"/>
+				<inertia
+				ixx="0.000002749" ixy="0.0"  ixz="0.0"
+				iyy="0.000007561" iyz="0.0"
+				izz="0.000005046" />
 			</inertial>
 		</link>
 		<gazebo reference="tibia_${side}${position}">
-			<material>Gazebo/DarkGrey</material>
+			<material>Gazebo/Black</material>
 		</gazebo>
 	</xacro:macro>
 <!-- Build robot model -->
-	<xacro:leg side="R" position="R" x="-0.065" y="-0.0325" angle="-${pi*3/4}" axis="1" />
+	<xacro:leg side="R" position="R" x="-0.065" y="-0.0325" angle="-${116.25*pi/180}" axis="1" />
 	<xacro:leg side="R" position="M" x="0.0" y="-0.0625" angle="-${pi/2}" axis="1" />
-	<xacro:leg side="R" position="F" x="0.065" y="-0.0325" angle="-${pi/4}" axis="1" />
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